File: hardware/adc.kicad_sch (KiCad schematic)
At the start: 6 parts, among them U2 AD8607

Commit message: Update PCB
Parts:
- removed U2: AD8607, AD8607:SO08, symbol AD8607:AD8607
- added U2: AD8603, Package_TO_SOT_SMD:TSOT-23-5, symbol Amplifier_Operational:AD8603
Connections:
- net +3V3: now also U2.5 (V+)
- net GND: now also U2.2 (V-)
- net SENS- renamed SENSOR
- net SENSOR: now also U2.3 (+)
- new net ADC: U2.1, U2.4 (-)
Other:
- note added: "BASINC SENSORU https://www.direnc.net/5-v-g14-0-12-mpa-hidrolik-suyaggaz-basinc-sensoru"
- moved on the sheet: C12, C13, D2, R8, R9
