File: hardware/damlama.kicad_sch (KiCad schematic)
At the start: 2 parts, among them J1 Conn_01x11_Male, J2 USB_B_Micro

Commit message: Update PCB
Parts:
- removed J1: Conn_01x11_Male, Connector_Phoenix_MSTB:PhoenixContact_MSTBA_2,5_11-G-5,08_1x11_P5.08mm_Horizontal, symbol Connector:Conn_01x11_Male
- added J1: COMM, Connector_Phoenix_MSTB:PhoenixContact_MSTBA_2,5_5-G-5,08_1x05_P5.08mm_Horizontal, symbol Connector:Screw_Terminal_01x05
- added J4: RELAY, Connector_Phoenix_MSTB:PhoenixContact_MSTBA_2,5_3-G-5,08_1x03_P5.08mm_Horizontal, symbol Connector:Screw_Terminal_01x03
- added J5: SENSOR, Connector_Phoenix_MSTB:PhoenixContact_MSTBA_2,5_3-G-5,08_1x03_P5.08mm_Horizontal, symbol Connector:Screw_Terminal_01x03
- added J6: POWER, Connector_Phoenix_MSTB:PhoenixContact_MSTBA_2,5_2-G-5,08_1x02_P5.08mm_Horizontal, symbol Connector:Screw_Terminal_01x02
Connections:
- net GND: now also J1.3 (Pin_3), J5.3 (Pin_3), J6.2 (Pin_2)
- net MCU/I2C_SCL: now also J1.4 (Pin_4)
- net MCU/I2C_SDA: now also J1.5 (Pin_5)
- net MCU/UART_RX: now also J1.2 (Pin_2)
- net MCU/UART_TX: now also J1.1 (Pin_1)
- net Power/VCC: now also J6.1 (Pin_1)
- new net +5V: J5.1 (Pin_1)
- new net ADC/SENSOR: J5.2 (Pin_2)
- new net Relay/RLIN: J4.3 (Pin_3)
- new net Relay/RLNC: J4.1 (Pin_1)
- new net Relay/RLNO: J4.2 (Pin_2)
Other:
- sheet ADC ports: added ADC, SENSOR; removed none
- sheet Relay ports: added RLCTL, RLIN, RLNC, RLNO; removed none
- note added: "INPUT: 9V/30V"
