File: hardware/mcu.kicad_sch (KiCad schematic)
At the start: 20 parts, among them J3 Conn_01x04_Male, SW1 SW_SPDT, U1 STM32F103C8Tx, Y1 16MHz

Commit message: Update PCB
Parts:
- removed R1, R2, R4: 1k5, Resistor_SMD:R_0402_1005Metric, symbol Device:R
- removed R3: 10k, Resistor_SMD:R_0402_1005Metric, symbol Device:R
- added R1, R2, R4: 1K5, Resistor_SMD:R_0603_1608Metric, symbol Device:R_Small
- added R3: 1K, Resistor_SMD:R_0603_1608Metric, symbol Device:R_Small
- U1: value STM32F103C8Tx -> STM32F103C8T6TR
Connections:
- net +3.3V: now also J3.3 (Pin_3), R1.1, R2.1, R4.1; no longer J3.1 (Pin_1)
- net I2C_SCL: now also R1.2
- net I2C_SDA: now also R2.2
- net SWCLK: now also J3.2 (Pin_2); no longer J3.3 (Pin_3)
- net SWDI0: now also J3.1 (Pin_1); no longer J3.2 (Pin_2)
- net SW_BOOT0: now also R3.1
- net USB_D+: now also R4.2
- net at U1.44 (BOOT0): now also R3.2
Other:
- moved on the sheet: J3
