File: hardware/power.kicad_sch (KiCad schematic)
At the start: 8 parts, among them U3 LD1086DT50TR, U4 AMS1117-3.3

Commit message: Update PCB
Changed lines of the file:
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@@
     (stroke (width 0) (type default) (color 0 0 0 0))
   )
-  (text "INPUT: 9V/30V" (at 90.17 80.01 0)
+  (text "INPUT: 9V/30V" (at 90.17 91.44 0)
     (effects (font (size 1.27 1.27)) (justify left bottom))
   )
