File: hardware/relay.kicad_sch (KiCad schematic)
At the start: 7 parts, among them Q1 BC847

Commit message: Update PCB
Parts:
- removed R7: 4K7, Resistor_SMD:R_0603_1608Metric, symbol Device:R
- removed RLY1: G5LE-14_DC12, digikey-footprints:Relay_THT_G5LE-14, symbol kanal-kapak-hardware-rescue:G5LE-14_DC12-dk_Power-Relays-Over-2-Amps
- removed RV1: Varistor, Varistor:RV_Disc_D7mm_W3.4mm_P5mm, symbol Device:Varistor
- added K1: SRD-05VDC-SL-C, Damlama:RELAY_SRD-05VDC-SL-C, symbol Damlama:SRD-05VDC-SL-C
Connections:
- net +12V is gone; now on an unnamed net: D1.1 (K)
- net GND: now also D1.2 (A)
- net RLIN: now also K1.COM
- net at Q1.3 (C): now also K1.A2; no longer D1.2 (A)
- new net +5V: K1.A1
- new net RLNC: K1.NC
- new net RLNO: K1.NO
- no-connect marks 1 -> 0
Other:
- moved on the sheet: D1, Q1, R5, R6
