File: hardware/gsm.kicad_sch (KiCad schematic)
At the start: 1 part, among them U3 SIM800L-CORE

Commit message: MCU BOOT0 mistake fixed
Parts:
- U3: now left out of the parts list
Changed lines of the file:
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@@
   )
   (symbol (lib_id "Damlama:SIM800L-CORE") (at 147.955 88.265 0) (unit 1)
-    (in_bom yes) (on_board yes) (dnp no) (fields_autoplaced)
+    (in_bom no) (on_board yes) (dnp no) (fields_autoplaced)
     (property "Reference" "U3" (at 148.59 76.2 0)
       (effects (font (size 1.27 1.27)))
